Commit message: feat(viewer): swap to V26 URDF + auto re-IK POSE_LIB for the new chain
V26 refactors the elbow: link3_elbow_connector becomes its own link
(link_elbow_connector) attached via joint_elbow_connector with
rpy=(0, π, 0), and joint_3 + everything downstream now hangs from
this flipped frame.  Net effect: joint_3's axis is inverted and the
chain offset changes — the V60 POSE_LIB joint values no longer reach
the same TCP world poses.

Strategy: keep the V60 joint values as TCP TARGETS, then re-IK each
pose against the V26 URDF at boot.

Implementation:
  - public/urdf/lexium_cobot.urdf is now V26 (with /meshes/v53/cobot+gripper/
    paths).  Old V60 file kept as lexium_cobot.v60.urdf.bak for reference.
  - POSE_LIB_V60 (frozen const) holds the original joints.
  - POSE_LIB (mutable) is initialised from V60 as a fallback, then
    overwritten at boot with V26 joints.
  - v60TcpWorldPose(): inline analytical FK of the V60 chain (joint
    origins, axes and the static rpy=(0,0,0.05) of joint_2 baked in).
    Produces the world {pos, quat} of tcp_link for any V60 joint vector
    — used to capture the TCP targets without needing to ship a second
    URDF for FK.
  - regeneratePoseLibForV26(): for each named pose, computes V60 TCP,
    seeds solveIK6D with V60 joints (close enough even with the j3
    flip) and stores the resulting V26 joints.  Returns the lib + any
    residual warnings (pos >5 mm or rot >2.9°).
  - Caching: results persisted in localStorage under
    schneider_v26_pose_lib_v1.  Boot loads cache if present, else polls
    for the cobot refs to be ready and regenerates once.
  - DEBUG/IK Solver section gains a status row (idle / cached / fresh
    / running / failed) and a blue "🔁 RE-IK all poses for V26" button
    that force-regenerates.  Warnings render in a scrollable amber box
    so the operator can see exactly which poses failed to converge
    cleanly.

The IK solver and animation player are unchanged — they read POSE_LIB
at runtime, so the cycle, pose-snap buttons and saved positions all
keep working with the regenerated joints.

Co-Authored-By: Claude Opus 4.7 <noreply@anthropic.com>

File: public/urdf/lexium_cobot.urdf (robot description, URDF)
Before this commit: robot lexium_cobot_with_final_gripper, 17 links, 16 joints
Links:
- added link link_elbow_connector; visual mesh filename=/meshes/v53/cobot/link3_elbow_connector.STL scale=0.001 0.001 0.001
- link link2_upper_arm: geometry visual mesh filename=/meshes/v53/cobot/link2_elbow_joint.STL scale=0.001 0.001 0.001; visual mesh filename=/meshes/v53/cobot/link2_shoulder_connector.STL scale=0.001 0.001 0.001
Joints:
- added joint joint_elbow_connector: type fixed, parent link2_upper_arm, child link_elbow_connector, origin xyz=0.001060 0.243625 0.119967 rpy=0 3.14159265359 0
- joint joint_3: origin xyz=-0.0015 0.2450 0.2258 rpy=0 0 0 -> xyz=0.002560 0.001375 0.113592 rpy=0 0 0; parent link2_upper_arm -> link_elbow_connector
