Commit message: fix(viewer): CAFI grasp uses V53 lateral_target frame + tracks disc rotation
Three CAFI issues called out by the user:

  1) Grasp offset: was driving the CAFI from tcp_link (the moving jaw
     tip), which sits ~4 cm offset from the V53 grasp centre.  The V53
     URDF defines cafi_lateral_target_frame on gripper_base at
     (0, 0.0166, 0.0768) for exactly this purpose.  Added that link to
     the cobot URDF.

  2) CAFI did not rotate with the disc.  Added on_fixture_1 / on_fixture_2
     states that copy the world pose of the turntable's cafi_part_X_link
     (parented to the fixture, which rotates with turntable_link).  Disc
     spin now carries the CAFI along automatically.

  3) Blue CAFIs were opaque markers.  Their material alpha dropped from
     1.0 to 0.22 — they stay as faint reference markers for the runtime
     CAFI to align to, without being mistaken for physical parts.

CafiMesh refactor:
  - Lifted cobotRobotRef + turntableRobotRef to the root via setter
    callbacks from Cobot / Turntable.
  - When attached, CafiMesh copies position AND quaternion from the
    URDF frame (so wrist orientation propagates to the workpiece) and
    uses the V53 lateral-grasp mesh offset (-0.213, +0.056, -0.023).
  - When static (conveyor / vision / bin) it uses an identity rotation
    and a centred mesh offset so the workpiece sits flat on the surface.

SEQUENCE updated: at_load → on_fixture_1 (disc rotation now carries the
held CAFI around the cycle naturally).

Co-Authored-By: Claude Opus 4.7 <noreply@anthropic.com>

File: dist/urdf/lexium_cobot.urdf (robot description, URDF)
Before this commit: robot lexium_cobot_with_final_gripper, 16 links, 15 joints
Links:
- added link cafi_lateral_target_frame
Joints:
- added joint cafi_lateral_target_fixed_joint: type fixed, parent gripper_base, child cafi_lateral_target_frame, origin xyz=0.000000 0.016600 0.076750 rpy=0 0 0

Commit message: feat: sync from DigitalTwinSchneider.zip source — diagram, models, SCADA tab
- Replace diagram.svg with up-to-date version from Sandbox (785 KB)
- Add 6 new turntable STLs to meshes/v53/turntable/ and dist/:
  fixture_with_switch_body, fixture_with_switch_sensor,
  limit_switch_base_tower_cut, limit_switch_tower_base_left/right,
  turntable_limit_switch_striker_cam
- Update lexium_cobot.urdf and turntable_rivet_cell_v43.urdf to Sandbox versions
- Add components/scada/ (ScadaView, scadaEngine, scadaConfig, scadaTypes,
  aiClient, useScada) — standalone SCADA dashboard with AI diagnosis mock
- Add SCADA tab to App.tsx nav (ScadaView)
- Rebuild dist/ with all updated assets

Co-Authored-By: Claude Sonnet 4.6 <noreply@anthropic.com>

File: dist/urdf/lexium_cobot.urdf (robot description, URDF)
Before this commit: robot lexium_cobot_with_final_gripper, 18 links, 17 joints
Joints:
- joint joint_1: limit lower=-3.14159 upper=3.14159 effort=50 velocity=3.14 -> lower=0 upper=6.28319 effort=50 velocity=3.14
